File: hardware/memory_test.kicad_pcb (KiCad board)
At the start: 2 copper layers, 90 x 47 mm, 29 parts, among them J1 Conn_01x15, J2 Conn_01x15

Commit message: Improve component location and reroute
Parts:
- added REF**: MountingHole_3.5mm_Pad, MountingHole:MountingHole_3.5mm_Pad, F.Cu at (159.0, 98.0)
- added REF**: MountingHole_3.5mm_Pad, MountingHole:MountingHole_3.5mm_Pad, F.Cu at (63.0, 46.0)
- added REF**: MountingHole_3.5mm_Pad, MountingHole:MountingHole_3.5mm_Pad, F.Cu at (63.0, 98.0)
- added REF**: MountingHole_3.5mm_Pad, MountingHole:MountingHole_3.5mm_Pad, F.Cu at (159.0, 46.0)
- U2: renamed from NAND - IS37SML01G1
- U3: renamed from NOR - MT25TL01GHBB
- U6: renamed from FRAM - CY15B108QN
- moved R6 20.0 mm to (154.0, 79.0)
- moved R25 18.9 mm to (135.0, 71.0), turned to 180 degrees
- moved R8 15.7 mm to (135.0, 69.0), turned to 180 degrees
- moved R19 15.3 mm to (110.0, 66.0), turned to 90 degrees
- moved R22 13.6 mm to (133.0, 79.0)
- moved R20 12.5 mm to (112.0, 56.0)
- moved C4 12.2 mm to (121.0, 84.0), turned to 180 degrees
- moved C3 11.0 mm to (135.0, 75.0), turned to 90 degrees
- moved R7 10.6 mm to (149.0, 83.0), turned to -90 degrees
- moved C6 9.36 mm to (121.0, 57.0)
- moved R3 8.96 mm to (116.0, 72.0), turned to 180 degrees
- moved C1 8.91 mm to (123.0, 70.0), turned to 180 degrees
- moved R21 6.85 mm to (150.0, 66.0)
- moved R4 5.58 mm to (136.0, 54.0)
- moved R11 5.47 mm to (110.6, 91.0), turned to 90 degrees
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- renumbered MRAM-MR25H40 to U1, EEPROM to U4
Routing:
- net +3V3: track 131.5 -> 63.0 mm, vias 14 -> 21
- net /MOSI: track 139.6 -> 98.1 mm, vias 2 -> 5
- net /CS_MT25_B: track 66.1 -> 39.5 mm, vias 3 -> 2
- net /CS_CY15: track 68.9 -> 48.7 mm, vias 0 -> 2
- net /MISO: track 117.1 -> 99.1 mm, vias 7 -> 8
- net GND: track 18.9 -> 2.00 mm, vias 8 -> 1
- net /CS_MT25_A: track 82.2 -> 69.0 mm
- net /HOLD: track 129.4 -> 117.0 mm, vias 5 -> 9
- net /SCK: track 117.3 -> 105.9 mm, vias 4 -> 5
- net /CS_IS37: track 66.8 -> 77.0 mm, vias 0 -> 2
- net /WP: track 141.8 -> 146.7 mm, vias 3 -> 6
- net /CS_M95: track 49.4 -> 45.6 mm
- net /CS_MR25: track 45.5 -> 42.7 mm, vias 0 -> 2
- added copper zone on B.Cu, net +3V3
- added copper zone on F.Cu, net GND
- removed copper zone on F.Cu, net +3V3
Other:
- board size 90 x 47 mm -> 108.9 x 65.9 mm
- board text added: "USB POR ESTE LADO"
- board text removed: "USB ↑"
