File: hardware/memory_test.kicad_sch (KiCad schematic)
At the start: 29 parts, among them J1 Conn_01x15, J2 Conn_01x15, U1 MR25H40, U2 IS37SML01G1, U3 MT25TL01GHBB, U4 M95M02-A125, U6 CY15B108QN

Commit message: Improve component location and reroute
Other:
- note added: "TODO: Mejorar las huellas para incluir el tamaño del chip y el indicador del pin 1"
- note added: "TODO: Revisar los WP con todos los pull ups para ver si es correcto poner uno en cada."
Changed lines of the file:
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@@
 		(title "Módulo de memorias")
 		(date "10/04/26")
-		(rev "v3")
+		(rev "0.3")
 		(company "TEIDESAT")
 		(comment 1 "Rubén Martín")
 	)
+	(text "TODO: Revisar los WP con todos los pull ups para ver si es correcto poner uno en cada."
+		(exclude_from_sim no)
+		(at 82.55 194.056 0)
+		(effects
+			(font
+				(size 1.27 1.27)
+			)
+		)
+	)
+	(text "TODO: Mejorar las huellas para incluir el tamaño del chip y el indicador del pin 1"
+		(exclude_from_sim no)
+		(at 82.55 199.136 0)
+		(effects
+			(font
+				(size 1.27 1.27)
+			)
+		)
+	)
 	(text_box "MRAM"
 		(exclude_from_sim no)
@@
 		)
 		(instances
-			(project "Memory V4"
+			(project "memory_test"
 				(path "/87b2155c-3559-46a9-b4e3-9f599b40938f"
 					(reference "R8")
@@
 		)
 		(instances
-			(project "Memory V4"
+			(project "memory_test"
 				(path "/87b2155c-3559-46a9-b4e3-9f599b40938f"
 					(reference "C4")
@@
 		)
 		(instances
-			(project "Memory V4"
+			(project "memory_test"
 				(path "/87b2155c-3559-46a9-b4e3-9f599b40938f"
 					(reference "R10")
@@
 		)
 		(instances
-			(project "Memory V4"
+			(project "memory_test"
 				(path "/87b2155c-3559-46a9-b4e3-9f599b40938f"
 					(reference "U4")
@@
 		)
 		(instances
-			(project "Memory V4"
+			(project "memory_test"
 				(path "/87b2155c-3559-46a9-b4e3-9f599b40938f"
 					(reference "R22")
@@
 		)
 		(instances
-			(project "Memory V4"
+			(project "memory_test"
 				(path "/87b2155c-3559-46a9-b4e3-9f599b40938f"
 					(reference "#PWR036")
@@
 		)
 		(instances
-			(project "Memory V4"
+			(project "memory_test"
 				(path "/87b2155c-3559-46a9-b4e3-9f599b40938f"
 					(reference "#PWR030")
@@
 		)
 		(instances
-			(project "Memory V4"
+			(project "memory_test"
 				(path "/87b2155c-3559-46a9-b4e3-9f599b40938f"
 					(reference "#PWR037")
@@
 		)
 		(instances
-			(project "Memory V4"
+			(project "memory_test"
 				(path "/87b2155c-3559-46a9-b4e3-9f599b40938f"
 					(reference "U6")
@@
 		)
 		(instances
-			(project "Memory V4"
+			(project "memory_test"
 				(path "/87b2155c-3559-46a9-b4e3-9f599b40938f"
 					(reference "#PWR023")
@@
 		)
 		(instances
-			(project "Memory V4"
+			(project "memory_test"
 				(path "/87b2155c-3559-46a9-b4e3-9f599b40938f"
 					(reference "#PWR029")
@@
 		)
 		(instances
-			(project "Memory V4"
+			(project "memory_test"
 				(path "/87b2155c-3559-46a9-b4e3-9f599b40938f"
 					(reference "U1")
@@
 		)
 		(instances
-			(project "Memory V4"
+			(project "memory_test"
 				(path "/87b2155c-3559-46a9-b4e3-9f599b40938f"
 					(reference "#PWR021")
@@
 		)
 		(instances
-			(project "Memory V4"
+			(project "memory_test"
 				(path "/87b2155c-3559-46a9-b4e3-9f599b40938f"
 					(reference "U2")
@@
 		)
 		(instances
-			(project "Memory V4"
+			(project "memory_test"
 				(path "/87b2155c-3559-46a9-b4e3-9f599b40938f"
 					(reference "#PWR05")
@@
 		)
 		(instances
-			(project "Memory V4"
+			(project "memory_test"
 				(path "/87b2155c-3559-46a9-b4e3-9f599b40938f"
 					(reference "#PWR08")
@@
 		)
 		(instances
-			(project "Memory V4"
+			(project "memory_test"
 				(path "/87b2155c-3559-46a9-b4e3-9f599b40938f"
 					(reference "R24")
@@
 		)
 		(instances
-			(project "Memory V4"
+			(project "memory_test"
 				(path "/87b2155c-3559-46a9-b4e3-9f599b40938f"
 					(reference "R9")
@@
 		)
 		(instances
-			(project "Memory V4"
+			(project "memory_test"
 				(path "/87b2155c-3559-46a9-b4e3-9f599b40938f"
 					(reference "#PWR06")
@@
 		)
 		(instances
-			(project "Memory V4"
+			(project "memory_test"
 				(path "/87b2155c-3559-46a9-b4e3-9f599b40938f"
 					(reference "#PWR027")
@@
 		)
 		(instances
-			(project "Memory V4"
+			(project "memory_test"
 				(path "/87b2155c-3559-46a9-b4e3-9f599b40938f"
 					(reference "R2")
@@
 		)
 		(instances
-			(project "Memory V4"
+			(project "memory_test"
 				(path "/87b2155c-3559-46a9-b4e3-9f599b40938f"
 					(reference "C2")
@@
 		)
 		(instances
-			(project "Memory V4"
+			(project "memory_test"
 				(path "/87b2155c-3559-46a9-b4e3-9f599b40938f"
 					(reference "#PWR09")
@@
 		)
 		(instances
-			(project "Memory V4"
+			(project "memory_test"
 				(path "/87b2155c-3559-46a9-b4e3-9f599b40938f"
 					(reference "R11")
@@
 		)
 		(instances
-			(project "Memory V4"
+			(project "memory_test"
 				(path "/87b2155c-3559-46a9-b4e3-9f599b40938f"
 					(reference "R21")
@@
 		)
 		(instances
-			(project "Memory V4"
+			(project "memory_test"
 				(path "/87b2155c-3559-46a9-b4e3-9f599b40938f"
 					(reference "#PWR018")
@@
 		)
 		(instances
-			(project "Memory V4"
+			(project "memory_test"
 				(path "/87b2155c-3559-46a9-b4e3-9f599b40938f"
 					(reference "#PWR015")
@@
 		)
 		(instances
-			(project "Memory V4"
+			(project "memory_test"
 				(path "/87b2155c-3559-46a9-b4e3-9f599b40938f"
 					(reference "U3")
@@
 		)
 		(instances
-			(project "Memory V4"
+			(project "memory_test"
 				(path "/87b2155c-3559-46a9-b4e3-9f599b40938f"
 					(reference "#PWR04")
@@
 		)
 		(instances
-			(project "Memory V4"
+			(project "memory_test"
 				(path "/87b2155c-3559-46a9-b4e3-9f599b40938f"
 					(reference "#PWR02")
@@
 		)
 		(instances
-			(project "Memory V4"
+			(project "memory_test"
 				(path "/87b2155c-3559-46a9-b4e3-9f599b40938f"
 					(reference "R7")
@@
 		)
 		(instances
-			(project "Memory V4"
+			(project "memory_test"
 				(path "/87b2155c-3559-46a9-b4e3-9f599b40938f"
 					(reference "#PWR017")
@@
 		)
 		(instances
-			(project "Memory V4"
+			(project "memory_test"
 				(path "/87b2155c-3559-46a9-b4e3-9f599b40938f"
 					(reference "C1")
@@
 		)
 		(instances
-			(project "Memory V4"
+			(project "memory_test"
 				(path "/87b2155c-3559-46a9-b4e3-9f599b40938f"
 					(reference "R6")
@@
 		)
 		(instances
-			(project "Memory V4"
+			(project "memory_test"
 				(path "/87b2155c-3559-46a9-b4e3-9f599b40938f"
 					(reference "#PWR020")
@@
 		)
 		(instances
-			(project "Memory V4"
+			(project "memory_test"
 				(path "/87b2155c-3559-46a9-b4e3-9f599b40938f"
 					(reference "#PWR031")
@@
 		)
 		(instances
-			(project "Memory V4"
+			(project "memory_test"
 				(path "/87b2155c-3559-46a9-b4e3-9f599b40938f"
 					(reference "#PWR010")
@@
 		)
 		(instances
-			(project "Memory V4"
+			(project "memory_test"
 				(path "/87b2155c-3559-46a9-b4e3-9f599b40938f"
 					(reference "#PWR019")
@@
 		)
 		(instances
-			(project "Memory V4"
+			(project "memory_test"
 				(path "/87b2155c-3559-46a9-b4e3-9f599b40938f"
 					(reference "R4")
@@
 		)
 		(instances
-			(project "Memory V4"
+			(project "memory_test"
 				(path "/87b2155c-3559-46a9-b4e3-9f599b40938f"
 					(reference "R19")
@@
 		)
 		(instances
-			(project "Memory V4"
+			(project "memory_test"
 				(path "/87b2155c-3559-46a9-b4e3-9f599b40938f"
 					(reference "#PWR07")
@@
 		)
 		(instances
-			(project "Memory V4"
+			(project "memory_test"
 				(path "/87b2155c-3559-46a9-b4e3-9f599b40938f"
 					(reference "#PWR024")
@@
 		)
 		(instances
-			(project "Memory V4"
+			(project "memory_test"
 				(path "/87b2155c-3559-46a9-b4e3-9f599b40938f"
 					(reference "J2")
@@
 		)
 		(instances
-			(project "Memory V4"
+			(project "memory_test"
 				(path "/87b2155c-3559-46a9-b4e3-9f599b40938f"
 					(reference "#PWR011")
@@
 		)
 		(instances
-			(project "Memory V4"
+			(project "memory_test"
 				(path "/87b2155c-3559-46a9-b4e3-9f599b40938f"
 					(reference "#PWR03")
@@
 		)
 		(instances
-			(project "Memory V4"
+			(project "memory_test"
 				(path "/87b2155c-3559-46a9-b4e3-9f599b40938f"
 					(reference "#PWR022")
@@
 		)
 		(instances
-			(project "Memory V4"
+			(project "memory_test"
 				(path "/87b2155c-3559-46a9-b4e3-9f599b40938f"
 					(reference "#PWR028")
@@
 		)
 		(instances
-			(project "Memory V4"
+			(project "memory_test"
 				(path "/87b2155c-3559-46a9-b4e3-9f599b40938f"
 					(reference "R25")
@@
 		)
 		(instances
-			(project "Memory V4"
+			(project "memory_test"
 				(path "/87b2155c-3559-46a9-b4e3-9f599b40938f"
 					(reference "#PWR026")
@@
 		)
 		(instances
-			(project "Memory V4"
+			(project "memory_test"
 				(path "/87b2155c-3559-46a9-b4e3-9f599b40938f"
 					(reference "C3")
@@
 		)
 		(instances
-			(project "Memory V4"
+			(project "memory_test"
 				(path "/87b2155c-3559-46a9-b4e3-9f599b40938f"
 					(reference "#PWR013")
@@
 		)
 		(instances
-			(project "Memory V4"
+			(project "memory_test"
 				(path "/87b2155c-3559-46a9-b4e3-9f599b40938f"
 					(reference "#PWR032")
@@
 		)
 		(instances
-			(project "Memory V4"
+			(project "memory_test"
 				(path "/87b2155c-3559-46a9-b4e3-9f599b40938f"
 					(reference "R1")
@@
 		)
 		(instances
-			(project "Memory V4"
+			(project "memory_test"
 				(path "/87b2155c-3559-46a9-b4e3-9f599b40938f"
 					(reference "#PWR016")
@@
 		)
 		(instances
-			(project "Memory V4"
+			(project "memory_test"
 				(path "/87b2155c-3559-46a9-b4e3-9f599b40938f"
 					(reference "C6")
@@
 		)
 		(instances
-			(project "Memory V4"
+			(project "memory_test"
 				(path "/87b2155c-3559-46a9-b4e3-9f599b40938f"
 					(reference "#PWR014")
@@
 		)
 		(instances
-			(project "Memory V4"
+			(project "memory_test"
 				(path "/87b2155c-3559-46a9-b4e3-9f599b40938f"
 					(reference "R5")
@@
 		)
 		(instances
-			(project "Memory V4"
+			(project "memory_test"
 				(path "/87b2155c-3559-46a9-b4e3-9f599b40938f"
 					(reference "R3")
@@
 		)
 		(instances
-			(project "Memory V4"
+			(project "memory_test"
 				(path "/87b2155c-3559-46a9-b4e3-9f599b40938f"
 					(reference "J1")
@@
 		)
 		(instances
-			(project "Memory V4"
+			(project "memory_test"
 				(path "/87b2155c-3559-46a9-b4e3-9f599b40938f"
 					(reference "#PWR025")
@@
 		)
 		(instances
-			(project "Memory V4"
+			(project "memory_test"
 				(path "/87b2155c-3559-46a9-b4e3-9f599b40938f"
 					(reference "R20")
